File: hardware/System_pomiaru_ciśnienia_Chemsilium.kicad_sch (KiCad schematic)
At the start: 7 parts, among them J1 PRESSURE_SENSOR_1, J3 PRESSURE_SENSOR_2, U1 ADS1115IDGS

Commit message: [feat] Initial test design for differential pressure sensor PCB
Initial PCB prototype for differential pressure measurement device.
Identified issues for future iterations:
- UART conflict between STM32 and Arduino Nano.
- Incorrect footprint for MPXM2202 sensor (pitch too small).
- Missing dedicated header for BMP280.
- Insufficient expansion pins (GPIOs for encoder).
- Integrated step-down converter requirement (current version lacks
onboard integration).
Parts:
- removed D4: 1N5819, Diode_THT:D_DO-41_SOD81_P10.16mm_Horizontal, symbol Diode:1N5819
- removed U1: ADS1115IDGS, Connector_PinSocket_2.54mm:PinSocket_1x10_P2.54mm_Vertical, symbol Analog_ADC:ADS1115IDGS
- added BZ1: Buzzer, Buzzer_Beeper:Buzzer_12x9.5RM7.6, symbol Device:Buzzer
- added C1: 330n, Capacitor_THT:CP_Radial_Tantal_D4.5mm_P2.50mm, symbol Device:C
- added C10, C11, C12, C13, C14, C15, C17, C3, C6, C9: 100n, Capacitor_SMD:C_0603_1608Metric_Pad1.08x0.95mm_HandSolder, symbol Device:C
- added C16, C4, C5: 10u, Capacitor_SMD:C_0805_2012Metric_Pad1.18x1.45mm_HandSolder, symbol Device:C
- added C2: 100u, Capacitor_THT:CP_Radial_D8.0mm_P3.80mm, symbol Device:C_Polarized
- added J2: Jack-DC, Connector_BarrelJack:BarrelJack_CUI_PJ-102AH_Horizontal, symbol Connector:Jack-DC
- added J4: Conn_01x08_Pin, Connector_PinHeader_2.54mm:PinHeader_2x04_P2.54mm_Vertical, symbol Connector:Conn_01x08_Pin
- added J5, J6: Conn_01x04_Pin, Connector_PinHeader_2.54mm:PinHeader_1x04_P2.54mm_Vertical, symbol Connector:Conn_01x04_Pin
- added R3, R4: 330, Resistor_THT:R_Axial_DIN0207_L6.3mm_D2.5mm_P2.54mm_Vertical, symbol Device:R
- added U1: L7805, Package_TO_SOT_THT:TO-220-3_Vertical, symbol Regulator_Linear:L7805
- added U2: ADS1220xPW, Package_SO:TSSOP-16_4.4x5mm_P0.65mm, symbol Analog_ADC:ADS1220xPW
- added U4: TXS0104EPW, Package_SO:TSSOP-14_4.4x5mm_P0.65mm, symbol Logic_LevelTranslator:TXS0104EPW
- added U5: STM32G030F6Px, Package_SO:TSSOP-20_4.4x6.5mm_P0.65mm, symbol MCU_ST_STM32G0:STM32G030F6Px
- added U7: AMS1117CD-3.3, Package_TO_SOT_SMD:TO-252-3_TabPin2, symbol Regulator_Linear:AMS1117CD-3.3
- R1: value 4k7 -> 10k; footprint Resistor_THT:R_Axial_DIN0207_L6.3mm_D2.5mm_P10.16mm_Horizontal -> Resistor_SMD:R_0603_1608Metric_Pad0.98x0.95mm_HandSolder
- R2: value 4k7 -> 330; footprint Resistor_THT:R_Axial_DIN0207_L6.3mm_D2.5mm_P10.16mm_Horizontal -> Resistor_THT:R_Axial_DIN0207_L6.3mm_D2.5mm_P2.54mm_Vertical
Connections:
- net 5V_PRESS_ANALOG is gone; now on net +5VCC: J1.3 (Pin_3), J3.3 (Pin_3)
- net GND: now also BZ1.2 (-), C1.2, C10.2, C11.2, C12.2, C13.2, C14.2, C15.2, C16.2, C17.2, C2.2, C3.2, C4.2, C5.2, C6.2, C9.2, J2.2, J4.7 (Pin_7), J4.8 (Pin_8), J5.1 (Pin_1), J6.1 (Pin_1), U1.2 (GND), U2.3 (CLK), U2.4 (DGND), U2.5 (AVSS), U2.8 (REFN0), U4.7 (GND), U5.5 (VSS), U7.1 (GND)
- net PRESS_A_1_N: now also U2.10 (AIN1)
- net PRESS_A_1_P: now also U2.11 (AIN0/REFP1)
- net PRESS_A_2_N: now also U2.6 (AIN3/REFN1)
- net PRESS_A_2_P: now also U2.7 (AIN2)
- net +5VCC: now reaches A1.30 (VIN)
- net +5VCC: now also C10.1, C11.1, C12.1, C14.1, C2.1, C3.1, J5.2 (Pin_2), U1.3 (OUT), U2.12 (AVDD), U2.9 (REFP0), U4.14 (V_{CCB})
- net LED_RED: now reaches A1.5 (D2)
- net LED_RED: now also R2.1
- net 3V3_MC_VCC: no longer names the net of A1.17 (3V3)
- net 5V_MC_VCC renamed +3VCC
- net +3VCC: now also C13.1, C15.1, C16.1, C5.1, C6.1, C9.1, J4.1 (Pin_1), U2.13 (DVDD), U4.1 (V_{CCA}), U4.8 (OE), U5.4 (VDD), U7.2 (VO); no longer R2.1
- net BUZZER_OUT renamed LED_YELLOW
- net LED_YELLOW: now also R3.1
- net LED_ERROR renamed LED_GREEN
- net LED_GREEN: now also R4.1
- net LED_WARNING renamed BUZZER
- net BUZZER: now also BZ1.1 (+)
- net SCL_ADC renamed LCD_SCL
- net LCD_SCL: now also J5.3 (Pin_3); no longer R1.2
- net SDA_ADC: no longer names the net of R2.2
- net SDA_ADC: now also J6.4 (Pin_4); no longer A1.23 (A4)
- net UART_PC_RX renamed UART_TX_MCU_5V
- net UART_TX_MCU_5V: now also U4.12 (B2)
- net UART_PC_TX renamed UART_RX_MCU_5V
- net UART_RX_MCU_5V: now also U4.13 (B1)
- new net: J6.2 (Pin_2), R4.2
- new net: J6.3 (Pin_3), R3.2
- new net +6V5: C1.1, C4.1, U1.1 (IN), U7.3 (VI)
- new net +9VCC: J2.1
- new net CS_ADC_3V3: U2.2 (~{CS}), U5.7 (PA0)
- new net DRDY_ADC_3V3: U2.14 (~{DRDY}), U5.15 (PA8/PB0/PB1/PB2)
- new net LCD_SDA: A1.23 (A4), J5.4 (Pin_4)
- new net MISO_ADC_3V3: U2.15 (DOUT/~{DRDY}), U5.13 (PA6)
- new net MOSI_ADC_3V3: U2.16 (DIN), U5.14 (PA7)
- new net NRST: C17.1, J4.4 (Pin_4), R1.2, U5.6 (NRST)
- new net SCK_ADC_3V3: U2.1 (SCLK), U5.8 (PA1)
- new net SWCLK: J4.2 (Pin_2), U5.19 (PA14/PA15)
- new net SWDIO: J4.3 (Pin_3), U5.18 (PA13)
- new net UART_RX_DEBUG: J4.6 (Pin_6)
- new net UART_RX_MCU_3V3: U4.2 (A1), U5.9 (PA2)
- new net UART_TX_DEBUG: J4.5 (Pin_5)
- new net UART_TX_MCU_3V3: U4.3 (A2), U5.10 (PA3)
Other:
- note added: "ADC - pressure reading"
- note added: "Barrel jack - power in"
- note added: "Debug"
- note added: "LCD connection"
- note added: "Linear stabilizators"
- note added: "Logic level stranslation"
- note added: "MCU's"
- note added: "Pressure sensors"
- note added: "Signaling - LED BUZZER"
- moved on the sheet: A1, J1, J3
